Commit message: Moves meshes and urdf files to seperate package

File: microstrain_inertial_description/urdf/microstrain_gq7.urdf.xacro (robot description, xacro)
@@ -9,5 +9,5 @@
         <origin xyz="0 0 0" rpy="1.5708 0 1.5708" />
         <geometry>
-          <mesh filename="package://microstrain_inertial_driver/meshes/microstrain_gq7.stl" scale="0.001 0.001 0.001" />
+          <mesh filename="package://microstrain_inertial_description/meshes/microstrain_gq7.stl" scale="0.001 0.001 0.001" />
         </geometry>
         <material name="microstrain_gq7_material"/>
